File: vco.kicad_pcb (KiCad board)
At the start: 2 copper layers, 60.6 x 232.6 mm, 122 parts, among them J1 EXP FM, J10 Square, J11 Conn_02x05_Odd_Even, J2 1V/OCT, J3 1V/OCT, J4 LIN FM, J5 PWM, J6 SYNC, J7 Sine, J8 Saw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

Commit message: checking all resistor values
Other:
- board text added: "Thermco 1K->"
Changed lines of the file:
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@@
     (effects (font (size 1 1) (thickness 0.15)) (justify mirror))
+  )
+  (gr_text "Thermco\n  1K->\n" (at 52.07 56.388 90) (layer "B.SilkS")
+    (effects (font (size 0.75 0.75) (thickness 0.1)) (justify mirror))
   )
   (gr_text "soft" (at 48.08 187.44) (layer "F.SilkS")

Commit message: v2 ready for manu
Parts:
- added D7: D_Dual_Series_AKC, Package_TO_SOT_SMD:SOT-23_Handsoldering, B.Cu at (45.3, 24.9)
- added D8: D_Dual_Series_AKC, Package_TO_SOT_SMD:SOT-23_Handsoldering, B.Cu at (45.3, 20.8)
- D1, D2, D3, D4, D5, D6: footprint Diode_SMD:D_SOD-323 -> Diode_SMD:D_SOD-323_HandSoldering
- H10: value pulse -> square
- H21: value SYNC HARDNESS -> sync hardness
- H8: value saw -> triangle
- H9: value triangle -> saw
- J8: value Saw -> locked
- RV11: value 220K -> 47K
- RV9: value 220K -> 10K
- moved J11 66.7 mm to (54.7, 18.3), turned to 180 degrees
- moved R10 54.3 mm to (76.8, 19.1)
- moved R11 54.1 mm to (76.8, 17.1)
- moved R18 53.9 mm to (76.8, 15.2)
- moved C8 52.6 mm to (70.5, 15.2)
- moved U2 52.3 mm to (71.1, 19.1)
- moved C4 52.1 mm to (65.4, 15.9)
- moved R21 51.6 mm to (65.4, 18.4)
- moved R15 51.1 mm to (65.4, 21.0)
- moved R13 51.1 mm to (43.8, 28.4), turned to -90 degrees
- moved R34 50.8 mm to (34.9, 72.4)
- moved R16 50.6 mm to (65.4, 23.5)
- moved R41 50.4 mm to (34.9, 76.8)
- moved R44 50.3 mm to (34.9, 78.7)
- moved R37 49.9 mm to (34.9, 74.3)
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Connections:
- D3 pad 1: Net-(D3-Pad1) -> Net-(D3-K)
- D3 pad 2: Net-(D3-Pad2) -> Net-(D3-A)
- D4 pad 1: Net-(D3-Pad2) -> Net-(D3-A)
- H21 pad 1: (no net) -> /face
- J11 pad 1: Net-(J11-Pad1) -> Net-(D8-common)
- J11 pad 10: Net-(J11-Pad10) -> Net-(D7-common)
- J11 pad 2: Net-(J11-Pad1) -> Net-(D8-common)
- J11 pad 9: Net-(J11-Pad10) -> Net-(D7-common)
- R12 pad 2: Net-(J11-Pad10) -> Net-(D7-K)
- R13 pad 1: Net-(J11-Pad1) -> Net-(D7-A)
- R30 pad 1: Net-(D3-Pad1) -> Net-(D3-K)
- R31 pad 2: Net-(R31-Pad2) -> Net-(U1D-+)
- R32 pad 2: Net-(R31-Pad2) -> Net-(U1D-+)
- R33 pad 1: Net-(R33-Pad1) -> Net-(U1D--)
- R34 pad 2: Net-(R31-Pad2) -> Net-(U1D-+)
- R35 pad 1: Net-(D3-Pad1) -> Net-(D3-K)
- U1 pad 12: GND -> Net-(U1D-+)
- U1 pad 13: Net-(D3-Pad1) -> Net-(U1D--)
- U1 pad 14: Net-(D3-Pad2) -> Net-(R39-Pad2)
- U3 pad 8: Net-(J11-Pad10) -> Net-(D7-K)
- U4 pad 2: Net-(J11-Pad1) -> Net-(D7-A)
- U4 pad 3: Net-(J11-Pad1) -> Net-(D7-A)
- U4 pad 6: Net-(J11-Pad1) -> Net-(D7-A)
- U4 pad 7: Net-(J11-Pad1) -> Net-(D7-A)
- U6 pad 12: Net-(R31-Pad2) -> GND
- U6 pad 13: Net-(R33-Pad1) -> Net-(D3-K)
- U6 pad 14: Net-(R39-Pad2) -> Net-(D3-A)
Routing:
- net GND: track 84.4 -> 225.1 mm
- net Net-(U1D-+): track 0.00 -> 105.1 mm, vias 0 -> 2
- net Net-(R31-Pad2): track 104.6 -> 0.00 mm, vias 4 -> 0
- net VSS: track 58.3 -> 126.3 mm
- net /TRIANGLE: track 106.5 -> 41.7 mm
- net /SINE: track 87.7 -> 34.6 mm
- net Net-(U2A--): track 22.2 -> 71.9 mm
- net Net-(J11-Pad1): track 49.4 -> 0.00 mm
- net /SQUARE: track 106.8 -> 59.1 mm
- net /CV1: track 12.7 -> 57.6 mm, vias 0 -> 1
- net /SAW: track 97.6 -> 52.8 mm
- net Net-(R27-Pad1): track 48.7 -> 90.5 mm, vias 4 -> 0
- net /COARSE: track 59.3 -> 17.6 mm, vias 2 -> 1
- net Net-(U6A--): track 58.7 -> 22.1 mm, vias 2 -> 0
- net /CV2: track 9.12 -> 44.1 mm, vias 0 -> 1
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- added copper zone on B.Cu, net /face
- added copper zone on F.Cu, net /face
- removed copper zone on B.Cu, net (none)
- removed copper zone on F.Cu, net (none)
Other:
- board size 60.6 x 232.6 mm -> 60.6 x 230.9 mm
- board text added: "thismatters/vco/v2"
- board text removed: "thismatters/vco/v1"

Commit message: v2 just about ready for manu
Parts:
- D7, D8: footprint Package_TO_SOT_SMD:SOT-23_Handsoldering -> Package_TO_SOT_SMD:SOT-23
- H1, H2: footprint Eurorack:Mech-AudioJack-Hole -> Eurorack:Mech-AudioJack-Hole-Input-Voct
- H3, H4, H5: footprint Eurorack:Mech-AudioJack-Hole -> Eurorack:Mech-AudioJack-Hole-Input-CV
- H6: footprint Eurorack:Mech-AudioJack-Hole -> Eurorack:Mech-AudioJack-Hole-Input-Clock
- Q1: value MMBFJ111 -> MMBFJ113
- R40: value 4.7K -> 8.2K
- R45: value 200K -> 180K
- R49: value 1.5K -> 1.2K
- RV1: value EXP FM LVL -> B25K
- RV2: value LIN FM LVL -> B25K
- RV3: value PWM LVL -> B25K
- RV4: value Tune -> B25K
- RV5: value Fine Tune -> B25K
- RV7: value PW -> B25K
- moved C2 27.0 mm to (49.5, 38.6), turned to 180 degrees
- moved RV9 23.5 mm to (72.7, 55.8), turned to 180 degrees
- moved RV10 14.4 mm to (78.3, 68.3)
- moved C3 12.5 mm to (39.5, 38.6), turned to 0 degrees
- moved C6 10.7 mm to (36.6, 20.3)
- moved C7 10.2 mm to (36.6, 28.6)
- moved R12 9.69 mm to (47.9, 26.0), turned to 180 degrees
- moved R13 6.25 mm to (47.9, 23.7), turned to 0 degrees
- moved H20 5.62 mm to (38.4, 119.8)
- moved H18 5.39 mm to (38.2, 242.3)
- moved D7 4.53 mm to (46.4, 29.3), turned to -90 degrees
- moved R51 4.31 mm to (49.6, 80.9)
- moved R44 4.01 mm to (37.5, 81.8)
- moved RV11 4.00 mm to (36.8, 50.9)
- moved R50 3.91 mm to (49.6, 78.5)
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Connections:
- D7 pad 1: Net-(D7-A) -> -12V
- D7 pad 2: Net-(D7-K) -> +12V
- D8 pad 1: Net-(D7-A) -> -12V
- D8 pad 2: Net-(D7-K) -> +12V
- J11 pad 1: Net-(D8-common) -> Net-(J11-Pin_1)
- J11 pad 10: Net-(D7-common) -> Net-(J11-Pin_10)
- J11 pad 2: Net-(D8-common) -> Net-(J11-Pin_1)
- J11 pad 9: Net-(D7-common) -> Net-(J11-Pin_10)
- R12 pad 1: +12V -> Net-(J11-Pin_10)
- R12 pad 2: Net-(D7-K) -> Net-(D7-common)
- R13 pad 1: Net-(D7-A) -> Net-(D8-common)
- R13 pad 2: -12V -> Net-(J11-Pin_1)
- U3 pad 8: Net-(D7-K) -> +12V
- U4 pad 2: Net-(D7-A) -> -12V
- U4 pad 3: Net-(D7-A) -> -12V
- U4 pad 6: Net-(D7-A) -> -12V
- U4 pad 7: Net-(D7-A) -> -12V
Routing:
- net GND: track 225.1 -> 166.5 mm, vias 8 -> 13
- net Net-(R22-Pad1): track 25.1 -> 4.42 mm, vias 1 -> 0
- net Net-(D7-A): track 19.4 -> 0.00 mm
- net Net-(R23-Pad1): track 20.3 -> 4.22 mm
- net Net-(D7-K): track 15.3 -> 0.00 mm
- net Net-(U1C--): track 10.7 -> 25.5 mm, vias 0 -> 1
- net +12V: track 165.7 -> 152.0 mm
- net VCC: track 122.6 -> 109.0 mm
- net VSS: track 126.3 -> 114.1 mm
- net Net-(U1B--): track 29.9 -> 41.7 mm
- net Net-(D5-K): track 24.3 -> 13.2 mm
- net Net-(J11-Pin_10): track 0.00 -> 10.3 mm
- net Net-(J11-Pin_1): track 0.00 -> 9.96 mm
- net -12V: track 149.2 -> 158.4 mm
- net Net-(D3-A): track 11.2 -> 19.9 mm
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Other:
- board size 60.6 x 230.9 mm -> 50.5 x 230.7 mm

Commit message: bom fixes
Parts:
- C2, C3: value 22U 50V -> 22u 50V
- R1: value 70K -> 68K
- R2, R38: value 50K -> 47K
Changed lines of the file:
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@@
         (effects (font (size 1 1) (thickness 0.15)) (justify mirror))
     )
-    (fp_text value "22U 50V" (at 1.25 -3.75) (layer "B.Fab")
+    (fp_text value "22u 50V" (at 1.25 -3.75) (layer "B.Fab")
         (effects (font (size 1 1) (thickness 0.15)) (justify mirror))
     )
@@
         (effects (font (size 1 1) (thickness 0.15)) (justify mirror))
     )
-    (fp_text value "50K" (at 0 -1.65 90) (layer "B.Fab")
+    (fp_text value "47K" (at 0 -1.65 90) (layer "B.Fab")
         (effects (font (size 1 1) (thickness 0.15)) (justify mirror))
     )
@@
         (effects (font (size 1 1) (thickness 0.15)) (justify mirror))
     )
-    (fp_text value "22U 50V" (at 1.25 -3.75) (layer "B.Fab")
+    (fp_text value "22u 50V" (at 1.25 -3.75) (layer "B.Fab")
         (effects (font (size 1 1) (thickness 0.15)) (justify mirror))
     )
@@
         (effects (font (size 1 1) (thickness 0.15)) (justify mirror))
     )
-    (fp_text value "70K" (at 0 -1.65 90) (layer "B.Fab")
+    (fp_text value "68K" (at 0 -1.65 90) (layer "B.Fab")
         (effects (font (size 1 1) (thickness 0.15)) (justify mirror))
     )
@@
         (effects (font (size 1 1) (thickness 0.15)) (justify mirror))
     )
-    (fp_text value "50K" (at 0 -1.65) (layer "B.Fab")
+    (fp_text value "47K" (at 0 -1.65) (layer "B.Fab")
         (effects (font (size 1 1) (thickness 0.15)) (justify mirror))
     )

Commit message: more BOM fixes
Parts:
- R14, R9: value 7.5K -> 27K
- RV1, RV2, RV3, RV4, RV5, RV7: value B25K -> B100K
Changed lines of the file:
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@@
         (effects (font (size 1 1) (thickness 0.15)))
     )
-    (fp_text value "B25K" (at 0 4.826 unlocked) (layer "F.Fab")
+    (fp_text value "B100K" (at 0 4.826 unlocked) (layer "F.Fab")
         (effects (font (size 1 1) (thickness 0.15)))
     )
@@
         (effects (font (size 1 1) (thickness 0.15)))
     )
-    (fp_text value "B25K" (at 0 4.826 unlocked) (layer "F.Fab")
+    (fp_text value "B100K" (at 0 4.826 unlocked) (layer "F.Fab")
         (effects (font (size 1 1) (thickness 0.15)))
     )
@@
         (effects (font (size 1 1) (thickness 0.15)))
     )
-    (fp_text value "B25K" (at 0 4.826 unlocked) (layer "F.Fab")
+    (fp_text value "B100K" (at 0 4.826 unlocked) (layer "F.Fab")
         (effects (font (size 1 1) (thickness 0.15)))
     )
@@
         (effects (font (size 1 1) (thickness 0.15)))
     )
-    (fp_text value "B25K" (at 0 4.826 unlocked) (layer "F.Fab")
+    (fp_text value "B100K" (at 0 4.826 unlocked) (layer "F.Fab")
         (effects (font (size 1 1) (thickness 0.15)))
     )
@@
         (effects (font (size 1 1) (thickness 0.15)))
     )
-    (fp_text value "B25K" (at 15.367 11.049 unlocked) (layer "F.Fab")
+    (fp_text value "B100K" (at 15.367 11.049 unlocked) (layer "F.Fab")
         (effects (font (size 1 1) (thickness 0.15)))
     )
@@
         (effects (font (size 1 1) (thickness 0.15)))
     )
-    (fp_text value "B25K" (at 0 4.826 unlocked) (layer "F.Fab")
+    (fp_text value "B100K" (at 0 4.826 unlocked) (layer "F.Fab")
         (effects (font (size 1 1) (thickness 0.15)))
     )
@@
     (descr "SOT, 3 Pin (https://www.jedec.org/system/files/docs/to-236h.pdf variant AB), generated with kicad-footprint-generator ipc_gullwing_generator.py")
     (tags "SOT TO_SOT_SMD")
-    (property "PartNum" "512-MMBFJ111")
+    (property "PartNum" "512-MMBFJ113")
     (property "Sheetfile" "vco.kicad_sch")
     (property "Sheetname" "")
@@
     (descr "SOIC, 14 Pin (JEDEC MS-012AB, https://www.analog.com/media/en/package-pcb-resources/package/pkg_pdf/soic_narrow-r/r_14.pdf), generated with kicad-footprint-generator ipc_gullwing_generator.py")
     (tags "SOIC SO")
-    (property "PartNum" "595-TL074CN")
+    (property "PartNum" "595-TL074CDR")
     (property "Sheetfile" "vco.kicad_sch")
     (property "Sheetname" "")
@@
         (effects (font (size 1 1) (thickness 0.15)) (justify mirror))
     )
-    (fp_text value "7.5K" (at 0 -1.65) (layer "B.Fab")
+    (fp_text value "27K" (at 0 -1.65) (layer "B.Fab")
         (effects (font (size 1 1) (thickness 0.15)) (justify mirror))
     )
@@
         (effects (font (size 1 1) (thickness 0.15)) (justify mirror))
     )
-    (fp_text value "7.5K" (at 0 -1.65) (layer "B.Fab")
+    (fp_text value "27K" (at 0 -1.65) (layer "B.Fab")
         (effects (font (size 1 1) (thickness 0.15)) (justify mirror))
     )
@@
     (descr "SO, 8 Pin (https://www.nxp.com/docs/en/data-sheet/PCF8523.pdf), generated with kicad-footprint-generator ipc_gullwing_generator.py")
     (tags "SO SO")
-    (property "PartNum" "595-OPA2137UA/2K5 --or-- 595-OPA2134UA/2K5")
+    (property "PartNum" "595-OPA2134UA/2K5")
     (property "Sheetfile" "vco.kicad_sch")
     (property "Sheetname" "")

Commit message: one last resistor value
Parts:
- R22: value 5K6 -> 2.2K
Changed lines of the file:
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@@
         (effects (font (size 1 1) (thickness 0.15)) (justify mirror))
     )
-    (fp_text value "5K6" (at 0 -1.65 90) (layer "B.Fab")
+    (fp_text value "2.2K" (at 0 -1.65 90) (layer "B.Fab")
         (effects (font (size 1 1) (thickness 0.15)) (justify mirror))
     )
