File: vco.kicad_pcb (KiCad board)
At the start: 2 copper layers, 50.5 x 230.7 mm, 124 parts, among them J1 EXP FM, J10 Square, J11 Conn_02x05_Odd_Even, J2 1V/OCT, J3 1V/OCT, J4 LIN FM, J5 PWM, J6 SYNC, J7 Sine, J8 locked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

Commit message: trimmer values
Parts:
- R22: value 2.2K -> 22K
- RV11: value 47K -> 50K
- RV6: value 220K -> 250K
- RV9: value 10K -> 100K
Changed lines of the file:
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@@
         (effects (font (size 1 1) (thickness 0.15)) (justify mirror))
     )
-    (fp_text value "220K" (at -2.54 -3.67) (layer "B.Fab")
+    (fp_text value "250K" (at -2.54 -3.67) (layer "B.Fab")
         (effects (font (size 1 1) (thickness 0.15)) (justify mirror))
     )
@@
         (effects (font (size 1 1) (thickness 0.15)) (justify mirror))
     )
-    (fp_text value "2.2K" (at 0 -1.65 90) (layer "B.Fab")
+    (fp_text value "22K" (at 0 -1.65 90) (layer "B.Fab")
         (effects (font (size 1 1) (thickness 0.15)) (justify mirror))
     )
@@
         (effects (font (size 1 1) (thickness 0.15)) (justify mirror))
     )
-    (fp_text value "47K" (at -2.54 -3.67 90) (layer "B.Fab")
+    (fp_text value "50K" (at -2.54 -3.67 90) (layer "B.Fab")
         (effects (font (size 1 1) (thickness 0.15)) (justify mirror))
     )
@@
     (descr "Potentiometer, vertical, Bourns 3296W, https://www.bourns.com/pdfs/3296.pdf")
     (tags "Potentiometer vertical Bourns 3296W")
-    (property "PartNum" "A-586")
+    (property "PartNum" "")
     (property "Sheetfile" "vco.kicad_sch")
     (property "Sheetname" "")
-    (property "Vendor" "Tayda")
+    (property "Vendor" "")
     (property "ki_description" "Trim-potentiometer")
     (property "ki_keywords" "resistor variable trimpot trimmer")
@@
         (effects (font (size 1 1) (thickness 0.15)) (justify mirror))
     )
-    (fp_text value "10K" (at -2.54 -3.67) (layer "B.Fab")
+    (fp_text value "100K" (at -2.54 -3.67) (layer "B.Fab")
         (effects (font (size 1 1) (thickness 0.15)) (justify mirror))
     )

Commit message: pcb updated for v2
Parts:
- moved R34 34.5 mm to (69.6, 87.6)
- moved R37 1.60 mm to (37.5, 75.6)
- moved R41 1.27 mm to (37.5, 78.2)
- moved R44 0.89 mm to (37.5, 80.9)
- moved D3 0.48 mm to (37.5, 73.1)
Routing:
- net Net-(U1D-+): track 112.1 -> 93.7 mm
- net VSS: track 114.1 -> 130.1 mm
- net VCC: track 109.0 -> 123.4 mm
- net GND: track 166.5 -> 164.4 mm
- net Net-(R27-Pad1): track 92.3 -> 90.5 mm
- net Net-(D3-A): track 19.9 -> 21.1 mm
- net /SINE: track 33.9 -> 32.7 mm
- net Net-(R41-Pad2): track 7.45 -> 6.44 mm
- net /SAW: track 50.2 -> 51.1 mm
- net Net-(D2-A): track 45.9 -> 45.1 mm
- net Net-(Q1-S): track 73.7 -> 72.9 mm
- net /TRIANGLE: track 40.9 -> 40.1 mm
- net Net-(D3-K): track 6.74 -> 7.35 mm
- net Net-(D2-K): track 16.0 -> 15.4 mm
- net -12V: track 158.4 -> 157.9 mm
Other:
- board text added: "1v/oct"
- board text added: "exp fm"
- board text added: "lin fm"
- board text added: "pwm"
- board text added: "sync"
