File: vco.kicad_sch (KiCad schematic)
At the start: 124 parts, among them J1 EXP FM, J10 Square, J11 Conn_02x05_Odd_Even, J2 1V/OCT, J3 1V/OCT, J4 LIN FM, J5 PWM, J6 SYNC, J7 Sine, J8 Saw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

Commit message: one last resistor value
Parts:
- R22: value 5K6 -> 2.2K
Changed lines of the file:
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@@
       (effects (font (size 1.27 1.27)) (justify right))
     )
-    (property "Value" "5K6" (at 176.53 114.3 90)
+    (property "Value" "2.2K" (at 176.53 114.3 90)
       (effects (font (size 1.27 1.27)) (justify right))
     )

Commit message: trimmer values
Parts:
- R22: value 2.2K -> 22K
- RV11: value 47K -> 50K
- RV6: value 220K -> 250K
- RV9: value 10K -> 100K; PartNum A-586 -> (none); Vendor Tayda -> (none)
Changed lines of the file:
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@@
   (symbol (lib_id "Device:R_Potentiometer_Trim") (at 182.88 116.84 90) (unit 1)
     (in_bom yes) (on_board yes) (dnp no) (fields_autoplaced)
-    (property "Reference" "RV9" (at 182.88 119.8864 90)
-      (effects (font (size 1.27 1.27)))
-    )
-    (property "Value" "10K" (at 182.88 122.4233 90)
+    (property "Reference" "RV9" (at 182.88 120.65 90)
+      (effects (font (size 1.27 1.27)))
+    )
+    (property "Value" "100K" (at 182.88 123.19 90)
       (effects (font (size 1.27 1.27)))
     )
@@
       (effects (font (size 1.27 1.27)) hide)
     )
-    (property "Vendor" "Tayda" (at 182.88 116.84 90)
-      (effects (font (size 1.27 1.27)) hide)
-    )
-    (property "PartNum" "A-586" (at 182.88 116.84 90)
+    (property "Vendor" "" (at 182.88 116.84 90)
+      (effects (font (size 1.27 1.27)) hide)
+    )
+    (property "PartNum" "" (at 182.88 116.84 90)
       (effects (font (size 1.27 1.27)) hide)
     )
@@
       (effects (font (size 1.27 1.27)) (justify right))
     )
-    (property "Value" "2.2K" (at 176.53 114.3 90)
+    (property "Value" "22K" (at 176.53 114.3 90)
       (effects (font (size 1.27 1.27)) (justify right))
     )
@@
   (symbol (lib_id "Device:R_Potentiometer_Trim") (at 265.43 17.78 270) (unit 1)
     (in_bom yes) (on_board yes) (dnp no) (fields_autoplaced)
-    (property "Reference" "RV11" (at 265.43 13.0642 90)
-      (effects (font (size 1.27 1.27)))
-    )
-    (property "Value" "47K" (at 265.43 15.6011 90)
+    (property "Reference" "RV11" (at 265.43 11.43 90)
+      (effects (font (size 1.27 1.27)))
+    )
+    (property "Value" "50K" (at 265.43 13.97 90)
       (effects (font (size 1.27 1.27)))
     )
@@
   (symbol (lib_id "Device:R_Potentiometer_Trim") (at 99.06 109.22 90) (unit 1)
     (in_bom yes) (on_board yes) (dnp no) (fields_autoplaced)
-    (property "Reference" "RV6" (at 99.06 112.2664 90)
-      (effects (font (size 1.27 1.27)))
-    )
-    (property "Value" "220K" (at 99.06 114.8033 90)
-      (effects (font (size 1.27 1.27)))
-    )
+    (property "Reference" "RV6" (at 99.06 113.03 90)
+      (effects (font (size 1.27 1.27)))
+    )
+    (property "Value" "250K" (at 99.06 115.57 90)
+      (effects (font (size 1.27 1.27)))
+    )
